Commit message: terminate homing based on time and not erro

File: tiago_pro_capsules.urdf (robot description, URDF)
Before this commit: robot tiago_pro, 74 links, 73 joints
Links:
- link gripper_left_fingertip_right_link: geometry collision cylinder length=0.110491 radius=0.045; collision sphere radius=0.045
